Commit message: fix(nav2): 修正 base_frame_id 为 base_link，并简化 TF 发布逻辑
- 将 base_frame_id 设置为 'base_link'，解决 AMCL 无法发布 map->odom 的问题
- 删除以下多余的静态 TF 发布节点：
  - footprint_publisher
  - velodyne_tf_publisher
  - lds_tf_publisher
  - map_to_odom_publisher
- 保留 robot_state_publisher 即可生成完整 TF 树
- auto_initial_pose.py 改为使用 odom → base_link 的变换，实现自动初始定位发布

File: ros2_ws/src/tongji_webot_bringup/resource/TurtleBot3Burger.urdf (robot description, URDF)
Before this commit: robot TurtleBot3Burger.urdf, 18 links, 17 joints
Joints:
- joint base_link_LDS-01_joint: origin xyz=-0.03 0 0.173 rpy=0 0 0 -> xyz=-0.03 0 0.083 rpy=0 0 0
- joint left wheel motor: limit effort=10 velocity=6.67 -> effort=10 velocity=50; origin xyz=0 0.08 0.033 rpy=-0.526852 -1.57079 -2.614737 -> xyz=0 0.08 0.033 rpy=-3.141591 0.542875 -0.000004
- joint right wheel motor: limit effort=10 velocity=6.67 -> effort=10 velocity=50; origin xyz=0 -0.08 0.033 rpy=0 -1.570796 0 -> xyz=0 -0.08 0.033 rpy=0 1.093886 0
